File: Effect/STM32/STM32.kicad_pcb (KiCad board)
At the start: 4 copper layers, 30 x 84 mm, 40 parts, among them J101 Conn_01x04_Pin, J102 Conn_01x04_Pin, J103 Conn_01x04_Pin, J104 Conn_01x04_Pin, J301 USB_C_Receptacle_USB2.0_16P, U101 LMR50410, U102 LP2985-5.0, U201 STM32H750VBTx, Y301 16MHz

Commit message: Update very incomplete STM32 board
I'm committing this partial work just to have the history, and because I
might use this as a starting point if I take up the mixed-mode thing in
the new GuitarPedal project.

It's almost certainly not worth saving, but you never know...

Signed-off-by: Linus Torvalds <torvalds@linux-foundation.org>
Parts:
- added C401: 1uF, Capacitor_SMD:C_0603_1608Metric, B.Cu at (135.9, 98.3)
- added C402: 1uF, Capacitor_SMD:C_0603_1608Metric, B.Cu at (135.9, 100.8)
- added R401: 220k, Resistor_SMD:R_0603_1608Metric, B.Cu at (135.9, 103.3)
- added R402: 1MEG, Resistor_SMD:R_0603_1608Metric, B.Cu at (135.9, 105.9)
- added R403: 1MEG, Resistor_SMD:R_0603_1608Metric, B.Cu at (135.9, 108.4)
- added R404: 220k, Resistor_SMD:R_0603_1608Metric, B.Cu at (135.9, 110.9)
- added R405: 220k, Resistor_SMD:R_0603_1608Metric, B.Cu at (135.9, 113.4)
- added R406: 220k, Resistor_SMD:R_0603_1608Metric, B.Cu at (135.9, 115.9)
- added U401: PCM3060, Package_SO:TSSOP-28_4.4x9.7mm_P0.65mm, B.Cu at (129.6, 102.7)
